File: PCB/Faikout/Faikout.kicad_sch (KiCad schematic)
At the start: 47 parts, among them J1 1x5, J2 TC2030-USB-NL, J3 Reset, Q1 BSS138PS, U1 TPS562246, U4 ESP32-S3-MINI-1

Commit message: LED loop for ATE
Connections:
- net GND: no longer U4.28 (GPIO33)
- net LEDO: now reaches D1.4 (O)
- net LEDO: now also U4.28 (GPIO33)
- no-connect marks 25 -> 24
Changed lines of the file:
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@@
 	)
 	(no_connect
-		(at 165.735 46.355)
-	)
-	(no_connect
 		(at 83.82 70.485)
 	)
@@
 		)
 	)
+	(global_label "LEDO"
+		(shape output)
+		(at 165.735 46.355 0)
+		(fields_autoplaced yes)
+		(effects
+			(font
+				(size 1.27 1.27)
+			)
+			(justify left)
+		)
+		(property "Intersheetrefs" "${INTERSHEET_REFS}"
+			(at 172.8436 46.355 0)
+			(effects
+				(font
+					(size 1.27 1.27)
+				)
+				(justify left)
+				(hide yes)
+			)
+		)
+	)
 	(global_label "BST"
 		(shape passive)
@@
 		)
 	)
+	(global_label "LEDO"
+		(shape input)
+		(at 114.3 70.485 0)
+		(fields_autoplaced yes)
+		(effects
+			(font
+				(size 1.27 1.27)
+			)
+			(justify left)
+		)
+		(property "Intersheetrefs" "${INTERSHEET_REFS}"
+			(at 121.4086 70.485 0)
+			(effects
+				(font
+					(size 1.27 1.27)
+				)
+				(justify left)
+				(hide yes)
+			)
+		)
+	)
 	(symbol
 		(lib_id "power:+3.3V")
@@
 					(unit 1)
 				)
-			)
-		)
-	)
-	(symbol
-		(lib_id "power:GND")
-		(at 114.3 70.485 90)
-		(unit 1)
-		(exclude_from_sim no)
-		(in_bom yes)
-		(on_board yes)
-		(dnp no)
-		(fields_autoplaced yes)
-		(property "Reference" "#PWR025"
-			(at 120.65 70.485 0)
-			(effects
-				(font
-					(size 1.27 1.27)
-				)
-				(hide yes)
-			)
-		)
-		(property "Value" "GND"
-			(at 117.475 70.485 90)
-			(effects
-				(font
-					(size 1.27 1.27)
-				)
-				(justify right)
-			)
-		)
-		(property "Footprint" ""
-			(at 114.3 70.485 0)
-			(effects
-				(font
-					(size 1.27 1.27)
-				)
-				(hide yes)
-			)
-		)
-		(property "Datasheet" ""
-			(at 114.3 70.485 0)
-			(effects
-				(font
-					(size 1.27 1.27)
-				)
-				(hide yes)
-			)
-		)
-		(property "Description" "Power symbol creates a global label with name \"GND\" , ground"
-			(at 114.3 70.485 0)
-			(effects
-				(font
-					(size 1.27 1.27)
-				)
-				(hide yes)
-			)
-		)
-		(pin "1"
-		)
-		(instances
-			(project "Faikin"
-				(path "/46c350bb-7de4-4e81-aafd-4af55e37aab0"
-					(reference "#PWR025")
-					(unit 1)
-				)

Commit message: Silkscreen fix
Connections:
- net LED is gone; now on net LEDO: D1.2 (I), U4.27 (GPIO47)
- net LEDO: no longer D1.4 (O), U4.28 (GPIO33)
- new net LEDI: D1.4 (O), U4.28 (GPIO33)
Changed lines of the file:
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@@
 		)
 	)
-	(global_label "LED"
+	(global_label "LEDO"
 		(shape input)
 		(at 158.115 46.355 180)
@@
 		)
 		(property "Intersheetrefs" "${INTERSHEET_REFS}"
-			(at 152.3369 46.355 0)
+			(at 151.0064 46.355 0)
 			(effects
 				(font
@@
 		)
 	)
-	(global_label "LEDO"
+	(global_label "LEDI"
 		(shape output)
 		(at 165.735 46.355 0)
@@
 		)
 		(property "Intersheetrefs" "${INTERSHEET_REFS}"
-			(at 172.8436 46.355 0)
+			(at 172.1179 46.355 0)
 			(effects
 				(font
@@
 		)
 	)
-	(global_label "LED"
+	(global_label "LEDO"
 		(shape output)
 		(at 114.3 103.505 0)
@@
 		)
 		(property "Intersheetrefs" "${INTERSHEET_REFS}"
-			(at 120.0781 103.505 0)
+			(at 121.4086 103.505 0)
 			(effects
 				(font
@@
 		)
 	)
-	(global_label "LEDO"
+	(global_label "LEDI"
 		(shape input)
 		(at 114.3 70.485 0)
@@
 		)
 		(property "Intersheetrefs" "${INTERSHEET_REFS}"
-			(at 121.4086 70.485 0)
-			(effects
-				(font
+			(at 120.6829 70.485 0)
+			(effects
+				(font

Commit message: footprint tidy
Parts:
- U1: footprint RevK:SOT-563 -> RevK:SOT-5x3-6
Changed lines of the file:
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@@
 			)
 		)
-		(property "Footprint" "RevK:SOT-563"
+		(property "Footprint" "RevK:SOT-5x3-6"
 			(at 81.28 177.8 0)
 			(effects
